File: Projet MOSH - Fonctionne.kicad_pcb (KiCad board)
At the start: 2 copper layers, 68.6 x 54.9 mm, 24 parts, among them J1 Power, J2 Digital/PWM, J3 Analog, J4 Digital/PWM, U2 LTC1050, U4 MCP41100

Commit message: Final
Other:
- board text added: "Fabre - Leroi"
Changed lines of the file:
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@@
   (gr_arc (start 100 46.5584) (mid 100.223185 46.019585) (end 100.762 45.7964)
     (stroke (width 0.15) (type solid)) (layer "Edge.Cuts"))
+  (gr_text "Fabre - Leroi\n" (at 119.5072 70.9932) (layer "B.Cu")
+    (effects (font (size 1.5 1.5) (thickness 0.3) bold) (justify left bottom mirror))
+  )
   (gr_text "ICSP" (at 164.897 72.06 90) (layer "Dwgs.User")
     (effects (font (size 1 1) (thickness 0.15)))
